File: Exkeylibur.kicad_pcb (KiCad board)
At the start: 2 copper layers, 120 x 101.1 mm, 25 parts, among them SW1 SW_Push, SW10 SW_Push, SW11 SW_Push, SW12 SW_Push, SW13 SW_Push, SW14 SW_Push, SW15 SW_Push, SW16 SW_Push, SW17 SW_Push, SW18 SW_Push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

Commit message: traces routed
Connections:
- PWR_SW1 pad 1: unconnected-(PWR_SW1-Pad1) -> (no net)
- U1 pad 1: unconnected-(U1-Pad1) -> switch6
- U1 pad 10: unconnected-(U1-Pad10) -> switch13
- U1 pad 11: unconnected-(U1-Pad11) -> switch7
- U1 pad 12: unconnected-(U1-Pad12) -> switch1
- U1 pad 13: unconnected-(U1-Pad13) -> switch8
- U1 pad 14: unconnected-(U1-Pad14) -> switch9
- U1 pad 15: unconnected-(U1-Pad15) -> switch10
- U1 pad 16: unconnected-(U1-Pad16) -> switch11
- U1 pad 17: unconnected-(U1-Pad17) -> switch12
- U1 pad 18: unconnected-(U1-Pad18) -> switch2
- U1 pad 19: unconnected-(U1-Pad19) -> switch3
- U1 pad 2: unconnected-(U1-Pad2) -> switch5
- U1 pad 20: unconnected-(U1-Pad20) -> switch4
- U1 pad 5: unconnected-(U1-Pad5) -> switch18
- U1 pad 6: unconnected-(U1-Pad6) -> switch17
- U1 pad 7: unconnected-(U1-Pad7) -> switch16
- U1 pad 8: unconnected-(U1-Pad8) -> switch15
- U1 pad 9: unconnected-(U1-Pad9) -> switch14
Routing:
- net switch14: track 0.00 -> 118.7 mm
- net switch15: track 0.00 -> 96.9 mm
- net switch8: track 0.00 -> 96.8 mm
- net switch2: track 0.00 -> 96.3 mm
- net switch16: track 0.00 -> 78.7 mm
- net switch3: track 0.00 -> 74.0 mm
- net switch9: track 0.00 -> 73.8 mm
- net switch17: track 0.00 -> 59.9 mm
- net switch4: track 0.00 -> 58.3 mm
- net switch10: track 0.00 -> 56.7 mm
- net switch5: track 0.00 -> 50.6 mm
- net switch18: track 0.00 -> 44.0 mm
- net switch13: track 0.00 -> 40.2 mm
- net Net-(RSW1-Pad1): track 0.00 -> 36.7 mm, vias 0 -> 1
- net switch11: track 0.00 -> 34.8 mm
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
Commit message: copper pour
Routing:
- net switch14: track 118.7 -> 120.1 mm
- added copper zone on B.Cu, net GND
- added copper zone on F.Cu, net GND
Changed lines of the file:
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@@
   (segment (start 95.954103 61.185821) (end 49.318979 61.185821) (width 0.25) (layer "F.Cu") (net 17))
   (segment (start 49.318979 61.185821) (end 48.389158 60.256) (width 0.25) (layer "F.Cu") (net 17))
-  (segment (start 37.699429 84.607421) (end 35.063737 84.607421) (width 0.25) (layer "F.Cu") (net 18))
-  (segment (start 72.973421 72.599421) (end 73.070425 72.696425) (width 0.25) (layer "F.Cu") (net 18))
-  (segment (start 41.400425 80.906425) (end 37.699429 84.607421) (width 0.25) (layer "F.Cu") (net 18))
-  (segment (start 73.070425 72.696425) (end 59.750425 72.696425) (width 0.25) (layer "F.Cu") (net 18))
-  (segment (start 35.063737 84.607421) (end 30.389158 89.282) (width 0.25) (layer "F.Cu") (net 18))
-  (segment (start 59.750425 72.696425) (end 51.540425 80.906425) (width 0.25) (layer "F.Cu") (net 18))
-  (segment (start 51.540425 80.906425) (end 41.400425 80.906425) (width 0.25) (layer "F.Cu") (net 18))
-  (segment (start 81.590425 81.216425) (end 98.860425 81.216425) (width 0.25) (layer "F.Cu") (net 18))
+  (segment (start 106.670425 89.026425) (end 113.580425 89.026425) (width 0.25) (layer "F.Cu") (net 18))
+  (segment (start 97.229465 79.585465) (end 106.670425 89.026425) (width 0.25) (layer "F.Cu") (net 18))
+  (segment (start 113.580425 89.026425) (end 128.322558 74.284292) (width 0.25) (layer "F.Cu") (net 18))
+  (segment (start 59.750425 72.696425) (end 72.980425 72.696425) (width 0.25) (layer "F.Cu") (net 18))
+  (segment (start 38.040425 79.046425) (end 53.400425 79.046425) (width 0.25) (layer "F.Cu") (net 18))
+  (segment (start 79.869465 79.585465) (end 97.229465 79.585465) (width 0.25) (layer "F.Cu") (net 18))
+  (segment (start 30.389158 86.697692) (end 38.040425 79.046425) (width 0.25) (layer "F.Cu") (net 18))
+  (segment (start 53.400425 79.046425) (end 59.750425 72.696425) (width 0.25) (layer "F.Cu") (net 18))
+  (segment (start 72.980425 72.696425) (end 79.869465 79.585465) (width 0.25) (layer "F.Cu") (net 18))
   (segment (start 128.322558 74.284292) (end 128.322558 73.406) (width 0.25) (layer "F.Cu") (net 18))
-  (segment (start 106.670425 89.026425) (end 113.580425 89.026425) (width 0.25) (layer "F.Cu") (net 18))
-  (segment (start 98.860425 81.216425) (end 106.670425 89.026425) (width 0.25) (layer "F.Cu") (net 18))
-  (segment (start 113.580425 89.026425) (end 128.322558 74.284292) (width 0.25) (layer "F.Cu") (net 18))
-  (segment (start 73.070425 72.696425) (end 81.590425 81.216425) (width 0.25) (layer "F.Cu") (net 18))
+  (segment (start 30.389158 89.282) (end 30.389158 86.697692) (width 0.25) (layer "F.Cu") (net 18))
   (segment (start 93.046 41.782) (end 84.389158 41.782) (width 0.25) (layer "F.Cu") (net 19))
   (segment (start 98.220425 43.896425) (end 95.160425 43.896425) (width 0.25) (layer "F.Cu") (net 19))
@@
   (segment (start 111.480425 74.323867) (end 111.480425 73.320427) (width 0.25) (layer "F.Cu") (net 20))
   (segment (start 105.920425 70.516425) (end 108.676423 70.516425) (width 0.25) (layer "F.Cu") (net 20))
+  (segment (start 80.889945 79.135945) (end 73.560425 71.806425) (width 0.25) (layer "F.Cu") (net 21))
+  (segment (start 53.70285 77.274) (end 48.389158 77.274) (width 0.25) (layer "F.Cu") (net 21))
   (segment (start 128.322558 71.824292) (end 111.720425 88.426425) (width 0.25) (layer "F.Cu") (net 21))
-  (segment (start 107.180425 88.426425) (end 98.330425 79.576425) (width 0.25) (layer "F.Cu") (net 21))
+  (segment (start 111.720425 88.426425) (end 107.180425 88.426425) (width 0.25) (layer "F.Cu") (net 21))
+  (segment (start 73.560425 71.806425) (end 59.170425 71.806425) (width 0.25) (layer "F.Cu") (net 21))
+  (segment (start 128.322558 70.866) (end 128.322558 71.824292) (width 0.25) (layer "F.Cu") (net 21))
   (segment (start 59.170425 71.806425) (end 53.70285 77.274) (width 0.25) (layer "F.Cu") (net 21))
-  (segment (start 98.330425 79.576425) (end 81.330425 79.576425) (width 0.25) (layer "F.Cu") (net 21))
-  (segment (start 128.322558 70.866) (end 128.322558 71.824292) (width 0.25) (layer "F.Cu") (net 21))
-  (segment (start 73.560425 71.806425) (end 59.170425 71.806425) (width 0.25) (layer "F.Cu") (net 21))
-  (segment (start 53.70285 77.274) (end 48.389158 77.274) (width 0.25) (layer "F.Cu") (net 21))
-  (segment (start 81.330425 79.576425) (end 73.560425 71.806425) (width 0.25) (layer "F.Cu") (net 21))
-  (segment (start 111.720425 88.426425) (end 107.180425 88.426425) (width 0.25) (layer "F.Cu") (net 21))
+  (segment (start 97.889945 79.135945) (end 80.889945 79.135945) (width 0.25) (layer "F.Cu") (net 21))
+  (segment (start 107.180425 88.426425) (end 97.889945 79.135945) (width 0.25) (layer "F.Cu") (net 21))
   (segment (start 113.102558 53.086) (end 114.012983 53.996425) (width 0.25) (layer "F.Cu") (net 23))
   (segment (start 116.940425 53.996425) (end 118.307925 53.996425) (width 0.25) (layer "F.Cu") (net 23))
@@
   (segment (start 122.907158 54.119692) (end 122.907158 53.891) (width 0.25) (layer "B.Cu") (net 23))
   (segment (start 116.940425 53.996425) (end 116.940425 54.148289) (width 0.25) (layer "B.Cu") (net 23))
+  (zone (net 3) (net_name "GND") (layer "F.Cu") (hatch edge 0.508)
+    (connect_pads (clearance 0.508))
+    (min_thickness 0.254) (filled_areas_thickness no)
+    (fill yes (thermal_gap 0.508) (thermal_bridge_width 0.508))
+    (polygon
+      (pts
+        (xy 149.330425 125.326425)
+        (xy 18.400425 122.976425)
+        (xy 20.250425 19.076425)
+        (xy 149.670425 18.906425)
+      )
+    )
+  )
+  (zone (net 3) (net_name "GND") (layer "B.Cu") (hatch edge 0.508)
+    (connect_pads (clearance 0.508))
+    (min_thickness 0.254) (filled_areas_thickness no)
+    (fill yes (thermal_gap 0.508) (thermal_bridge_width 0.508))
+    (polygon
+      (pts
+        (xy 153.680425 130.356425)
+        (xy 15.860425 130.146425)
+        (xy 15.660425 16.106425)
+        (xy 155.760425 15.896425)
+      )
+    )
+  )
 )
